Commit message: Add rocker_to_frame_connector

File: urdf/Mars-Rover-URDF.urdf (robot description, URDF)
Before this commit: robot Mars-Rover-URDF, 1 links, 0 joints
Links:
- added link rocker_to_frame_connector, mass 0.017817; collision mesh filename=package://Mars-Rover-URDF/meshes/rocker_to_frame_connector.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; visual mesh filename=package://Mars-Rover-URDF/meshes/rocker_to_frame_connector.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
- link base_link: mass 1.5948 -> 1.59483552
Joints:
- added joint rocker_to_frame_connector_joint: type fixed, parent base_link, child rocker_to_frame_connector, origin xyz=0.0079 -0.003 0 rpy=0 0 0, axis 0 0 0

Commit message: right_rocker_pivot_crosslink

File: urdf/Mars-Rover-URDF.urdf (robot description, URDF)
Before this commit: robot Mars-Rover-URDF, 2 links, 1 joints
Links:
- added link right_rocker_pivot_crosslink, mass 7.0894; collision mesh filename=package://Mars-Rover-URDF/meshes/right_rocker_pivot_crossli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; visual mesh filename=package://Mars-Rover-URDF/meshes/right_rocker_pivot_crossli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
- link rocker_to_frame_connector: mass 0.017817 -> 0.0178174846110633
Joints:
- added joint right_rocker_pivot: type continuous, parent rocker_to_frame_connector, child right_rocker_pivot_crosslink, origin xyz=-0.0019 -0.2008 0.1732 rpy=0 0.42268 0, axis 0 1 0
- joint rocker_to_frame_connector_joint: origin xyz=0.0079 -0.003 0 rpy=0 0 0 -> xyz=0.00789999999999999 -0.00300000000000007 0 rpy=0 0 0

Commit message: Redo base link starting from updated assembly

File: urdf/Mars-Rover-URDF.urdf (robot description, URDF)
Before this commit: robot Mars-Rover-URDF, 3 links, 2 joints
Links:
- removed link right_rocker_pivot_crosslink
- removed link rocker_to_frame_connector
- link base_link: mass 1.59483552 -> 1.5948
Joints:
- removed joint right_rocker_pivot
- removed joint rocker_to_frame_connector_joint

Commit message: Add xbar top frame

File: urdf/Mars-Rover-URDF.urdf (robot description, URDF)
Before this commit: robot Mars-Rover-URDF, 1 links, 0 joints
Links:
- added link xbar_top_frame, mass 0.18097; collision mesh filename=package://Mars-Rover-URDF/meshes/xbar_top_frame.STL; visual mesh filename=package://Mars-Rover-URDF/meshes/xbar_top_frame.STL
- link base_link: mass 1.5948 -> 1.59483552
Joints:
- added joint xbar_to_chassis_joint: type fixed, parent base_link, child xbar_top_frame, origin xyz=0.016543 -0.00062631 0.024582 rpy=0 0 0, axis 0 0 0

Commit message: Add rocker_to_frame_mount_left link/joint

File: urdf/Mars-Rover-URDF.urdf (robot description, URDF)
Before this commit: robot Mars-Rover-URDF, 2 links, 1 joints
Links:
- added link rocker_to_frame_mount_left, mass 0.017817; collision mesh filename=package://Mars-Rover-URDF/meshes/rocker_to_frame_mount_left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; visual mesh filename=package://Mars-Rover-URDF/meshes/rocker_to_frame_mount_left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
- link xbar_top_frame: mass 0.18097 -> 0.180967186857142
Joints:
- added joint rocker_to_frame_mount_left_joint: type fixed, parent xbar_top_frame, child rocker_to_frame_mount_left, origin xyz=0 0 0 rpy=0 0 3.1416, axis 0 0 0
- joint xbar_to_chassis_joint: origin xyz=0.016543 -0.00062631 0.024582 rpy=0 0 0 -> xyz=0.0165427022776656 -0.000626311138720845 0.0245815452491259 rpy=0 0 0

Commit message: Add left rocker link/joint

File: urdf/Mars-Rover-URDF.urdf (robot description, URDF)
Before this commit: robot Mars-Rover-URDF, 3 links, 2 joints
Links:
- added link left_rocker, mass 0.2386; collision mesh filename=package://Mars-Rover-URDF/meshes/left_rocker.STL; visual mesh filename=package://Mars-Rover-URDF/meshes/left_rocker.STL
- link rocker_to_frame_mount_left: mass 0.017817 -> 0.0178174846110633
Joints:
- added joint left_rocker_joint: type continuous, parent rocker_to_frame_mount_left, child left_rocker, origin xyz=-0.0019 -0.2008 0.1732 rpy=0 0.20522 0, axis 0 1 0
- joint rocker_to_frame_mount_left_joint: origin xyz=0 0 0 rpy=0 0 3.1416 -> xyz=0 0 0 rpy=0 0 3.14159265358979
- joint xbar_to_chassis_joint: origin xyz=0.0165427022776656 -0.000626311138720845 0.0245815452491259 rpy=0 0 0 -> xyz=0.0176427022776656 -0.000626311138720845 0.0245815452491259 rpy=0 0 0

Commit message: Add left rocker wheel strut

File: urdf/Mars-Rover-URDF.urdf (robot description, URDF)
Before this commit: robot Mars-Rover-URDF, 4 links, 3 joints
Links:
- added link left_rocker_wheel_strut, mass 0.2153; collision mesh filename=package://Mars-Rover-URDF/meshes/left_rocker_wheel_strut.STL; visual mesh filename=package://Mars-Rover-URDF/meshes/left_rocker_wheel_strut.STL
- link left_rocker: mass 0.2386 -> 0.238601333424936
Joints:
- added joint left_rocker_wheel_strut_joint: type continuous, parent left_rocker, child left_rocker_wheel_strut, origin xyz=-0.4365 -0.01475 -0.061101 rpy=0 0 3.0493, axis 0 0 1
- joint left_rocker_joint: origin xyz=-0.0019 -0.2008 0.1732 rpy=0 0.20522 0 -> xyz=0.00189999999999785 -0.2008 0.173199999999999 rpy=0 0.205218691223717 0
- joint xbar_to_chassis_joint: origin xyz=0.0176427022776656 -0.000626311138720845 0.0245815452491259 rpy=0 0 0 -> xyz=0.0214427022776656 -0.000626311138720928 0.024581545249126 rpy=0 0 0

Commit message: Add left front wheel

File: urdf/Mars-Rover-URDF.urdf (robot description, URDF)
Before this commit: robot Mars-Rover-URDF, 5 links, 4 joints
Links:
- added link front_left_wheel, mass 0.59276; collision mesh filename=package://Mars-Rover-URDF/meshes/front_left_wheel.STL; visual mesh filename=package://Mars-Rover-URDF/meshes/front_left_wheel.STL
- link left_rocker_wheel_strut: mass 0.2153 -> 0.215297840696796
Joints:
- added joint front_left_wheel_joint: type continuous, parent left_rocker_wheel_strut, child front_left_wheel, origin xyz=0.00037346 3.3919E-05 -0.22684 rpy=-3.0812 0.26072 -2.8204, axis 0.22081 -0.97532 0
- joint left_rocker_wheel_strut_joint: origin xyz=-0.4365 -0.01475 -0.061101 rpy=0 0 3.0493 -> xyz=-0.436500004239615 -0.01475 -0.0611007329555057 rpy=0 0 3.04933024079565

Commit message: Add completed left bogie and wheels

File: urdf/Mars-Rover-URDF.urdf (robot description, URDF)
Before this commit: robot Mars-Rover-URDF, 6 links, 5 joints
Links:
- added link front_back_wheel, mass 0.59276; collision mesh filename=package://Mars-Rover-URDF/meshes/front_back_wheel.STL; visual mesh filename=package://Mars-Rover-URDF/meshes/front_back_wheel.STL
- added link left_bogie, mass 0.191498434857371; collision mesh filename=package://Mars-Rover-URDF/meshes/left_bogie.STL; visual mesh filename=package://Mars-Rover-URDF/meshes/left_bogie.STL
- added link left_bogie_wheel_strut, mass 0.215297841060573; collision mesh filename=package://Mars-Rover-URDF/meshes/left_bogie_wheel_strut.STL; visual mesh filename=package://Mars-Rover-URDF/meshes/left_bogie_wheel_strut.STL
- added link left_middle_wheel, mass 0.592760238512045; collision mesh filename=package://Mars-Rover-URDF/meshes/left_middle_wheel.STL; visual mesh filename=package://Mars-Rover-URDF/meshes/left_middle_wheel.STL
- link front_left_wheel: mass 0.59276 -> 0.592760238512046
Joints:
- added joint front_back_wheel_joint: type continuous, parent left_bogie_wheel_strut, child front_back_wheel, origin xyz=0.00037346 3.3919E-05 -0.16213 rpy=-0.54091 1.1566 -0.49012, axis 0.22081 -0.97532 0
- added joint left_bogie_joint: type continuous, parent left_rocker, child left_bogie, origin xyz=0.191978071510022 0 -0.130588977226116 rpy=0 -0.316495515015275 0, axis 0 1 0
- added joint left_bogie_wheel_strut_joint: type continuous, parent left_bogie, child left_bogie_wheel_strut, origin xyz=0.282426325346583 -0.014875000000001 0 rpy=0 0 2.92666748379435, axis 0 0 1
- added joint left_middle_wheel_joint: type continuous, parent left_bogie, child left_middle_wheel, origin xyz=-0.220157828209466 0 -0.145023978949895 rpy=-3.06072262662052 0.342728964216389 0.236649656298727, axis 0.220811799511535 -0.975316435418002 0
- joint front_left_wheel_joint: axis 0.22081 -0.97532 0 -> 0.220811799511534 -0.975316435418002 0; origin xyz=0.00037346 3.3919E-05 -0.22684 rpy=-3.0812 0.26072 -2.8204 -> xyz=0.000373462813278103 3.39194206695481E-05 -0.226836767044501 rpy=-3.08115374387749 0.26072091977244 -2.82044418134632
- joint rocker_to_frame_mount_left_joint: origin xyz=0 0 0 rpy=0 0 3.14159265358979 -> xyz=0.0038 0 0 rpy=0 0 3.14159265358979
- joint xbar_to_chassis_joint: origin xyz=0.0214427022776656 -0.000626311138720928 0.024581545249126 rpy=0 0 0 -> xyz=0.0176427022776656 -0.000626311138720845 0.0245815452491259 rpy=0 0 0

Commit message: Add rocker to frame mount right

File: urdf/Mars-Rover-URDF.urdf (robot description, URDF)
Before this commit: robot Mars-Rover-URDF, 10 links, 9 joints
Links:
- added link rocker_to_frame_mount_right, mass 0.017817; collision mesh filename=package://Mars-Rover-URDF/meshes/rocker_to_frame_mount_righ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; visual mesh filename=package://Mars-Rover-URDF/meshes/rocker_to_frame_mount_righ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
- link left_middle_wheel: mass 0.592760238512045 -> 0.59276
- link left_rocker_wheel_strut: mass 0.215297840696796 -> 0.2153
- link xbar_top_frame: mass 0.180967186857142 -> 0.18097
Joints:
- added joint rocker_to_frame_mount_right_joint: type fixed, parent xbar_top_frame, child rocker_to_frame_mount_right, origin xyz=0 0 0 rpy=0 0 0, axis 0 0 0

Commit message: Add right rocker

File: urdf/Mars-Rover-URDF.urdf (robot description, URDF)
Before this commit: robot Mars-Rover-URDF, 11 links, 10 joints
Links:
- added link right_front_wheel, mass 0.59276; collision mesh filename=package://Mars-Rover-URDF/meshes/right_front_wheel.STL; visual mesh filename=package://Mars-Rover-URDF/meshes/right_front_wheel.STL
- added link right_rocker, mass 0.23860136190612; collision mesh filename=package://Mars-Rover-URDF/meshes/right_rocker.STL; visual mesh filename=package://Mars-Rover-URDF/meshes/right_rocker.STL
- added link right_rocker_wheel_strut, mass 0.215297840693502; collision mesh filename=package://Mars-Rover-URDF/meshes/right_rocker_wheel_strut.S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; visual mesh filename=package://Mars-Rover-URDF/meshes/right_rocker_wheel_strut.S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
- link front_back_wheel: mass 0.59276 -> 0.592760238512045
- link front_left_wheel: mass 0.592760238512046 -> 0.592760238512045
- link left_middle_wheel: mass 0.59276 -> 0.592760238512045
- link left_rocker_wheel_strut: mass 0.2153 -> 0.215297840696796
- link rocker_to_frame_mount_right: mass 0.017817 -> 0.0178174846110633
- link xbar_top_frame: mass 0.18097 -> 0.180967186857142
Joints:
- added joint right_front_wheel_joint: type continuous, parent right_rocker, child right_front_wheel, origin xyz=-0.4365 0.01525 -0.16809 rpy=-3.1408 0.0034092 0.22265, axis 0.0034092 0.00077185 0.99999
- added joint right_rocker_joint: type continuous, parent rocker_to_frame_mount_right, child right_rocker, origin xyz=0.00190000000000082 -0.2008 0.173199999999998 rpy=0 -0.255302519881884 3.14159265358965, axis 0 1 0
- added joint right_rocker_wheel_strut_joint: type continuous, parent right_rocker, child right_rocker_wheel_strut, origin xyz=-0.436500004239613 0.0152499999999373 -0.0329909201580134 rpy=0 0 2.91894591666021, axis 0 0 1
- joint front_back_wheel_joint: axis 0.22081 -0.97532 0 -> 0.220811799511534 -0.975316435418002 0; origin xyz=0.00037346 3.3919E-05 -0.16213 rpy=-0.54091 1.1566 -0.49012 -> xyz=0.000373462813279157 3.39194206695204E-05 -0.162133741980369 rpy=-0.540911922792394 1.15655588476994 -0.490122742369759

Commit message: Add completed right bogie, strut, and wheels

File: urdf/Mars-Rover-URDF.urdf (robot description, URDF)
Before this commit: robot Mars-Rover-URDF, 14 links, 13 joints
Links:
- added link right_back_wheel, mass 0.592760238512046; collision mesh filename=package://Mars-Rover-URDF/meshes/right_back_wheel.STL; visual mesh filename=package://Mars-Rover-URDF/meshes/right_back_wheel.STL
- added link right_bogie, mass 0.191498434460467; collision mesh filename=package://Mars-Rover-URDF/meshes/right_bogie.STL; visual mesh filename=package://Mars-Rover-URDF/meshes/right_bogie.STL
- added link right_bogie_wheel_strut, mass 0.215297868113389; collision mesh filename=package://Mars-Rover-URDF/meshes/right_bogie_wheel_strut.STL; visual mesh filename=package://Mars-Rover-URDF/meshes/right_bogie_wheel_strut.STL
- added link right_middle_wheel, mass 0.592760238512045; collision mesh filename=package://Mars-Rover-URDF/meshes/right_middle_wheel.STL; visual mesh filename=package://Mars-Rover-URDF/meshes/right_middle_wheel.STL
- link front_left_wheel: mass 0.592760238512045 -> 0.592760238512046
- link right_front_wheel: mass 0.59276 -> 0.592760238512045
Joints:
- added joint right_back_wheel_joint: type continuous, parent right_bogie_wheel_strut, child right_back_wheel, origin xyz=0.00012191 2.7601E-05 -0.16213 rpy=0.23717 -0.80393 3.0404, axis 0.22081 -0.97532 0
- added joint right_bogie_joint: type continuous, parent right_rocker, child right_bogie, origin xyz=0.19198 0 -0.13059 rpy=0 0.14041 0, axis 0 1 0
- added joint right_bogie_wheel_strut_joint: type continuous, parent right_bogie, child right_bogie_wheel_strut, origin xyz=0.282426325346583 0.0146249999999995 0 rpy=0 0 3.1072058885597, axis 0 0 1
- added joint right_middle_wheel_joint: type continuous, parent right_bogie, child right_middle_wheel, origin xyz=-0.22016 0 -0.14502 rpy=-0.12179 0.49252 2.8883, axis 0.22081 -0.97532 0
- joint right_front_wheel_joint: origin xyz=-0.4365 0.01525 -0.16809 rpy=-3.1408 0.0034092 0.22265 -> xyz=0 0 -0.1351 rpy=-3.1408 0.0034092 -2.6963; parent right_rocker -> right_rocker_wheel_strut
